File: hardware/time-marker/time-marker.kicad_sch (KiCad schematic)
At the start: 77 parts, among them J1 Screw_Terminal_01x02, J10 Conn_01x02_Pin, J2 Conn_01x03_Pin, J3 Conn_01x05_Socket, J4 DE9_Plug_MountingHoles, J5 Conn_01x03_Pin, J6 Conn_02x03_Odd_Even, J7 Conn_02x03_Odd_Even, J8 Conn_01x03_Pin, J9 Conn_01x02_Pin, U2 ATmega8-16P, U3 MAX232, Y1 Crystal

Commit message: Added images and readme
Other:
- note added: "Grid frequency"
- note added: "Power supply"
- note added: "marker generator"
- note added: "optional RS232 port"
- note added: "optional lights and switches"
Changed lines of the file:
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@@
+		)
+	)
+	(polyline
+		(pts
+			(xy 107.95 55.88) (xy 107.95 90.17)
+		)
+		(stroke
+			(width 0)
+			(type default)
 		)
 	)
@@
 		)
 	)
+	(polyline
+		(pts
+			(xy 158.75 11.43) (xy 158.75 90.17)
+		)
+		(stroke
+			(width 0)
+			(type default)
+		)
+	)
 	(wire
 		(pts
@@
 		)
 	)
+	(polyline
+		(pts
+			(xy 11.43 34.29) (xy 107.95 34.29)
+		)
+		(stroke
+			(width 0)
+			(type default)
+		)
+	)
 	(wire
 		(pts
@@
 		)
 	)
+	(polyline
+		(pts
+			(xy 222.25 72.39) (xy 177.8 72.39)
+		)
+		(stroke
+			(width 0)
+			(type default)
+		)
+	)
 	(wire
 		(pts
@@
 		)
 	)
+	(polyline
+		(pts
+			(xy 177.8 72.39) (xy 177.8 166.37)
+		)
+		(stroke
+			(width 0)
+			(type default)
+		)
+	)
 	(wire
 		(pts
@@
 	(polyline
 		(pts
+			(xy 222.25 41.91) (xy 222.25 72.39)
+		)
+		(stroke
+			(width 0)
+			(type default)
+		)
+	)
+	(polyline
+		(pts
 			(xy 154.94 142.24) (xy 157.48 142.24)
 		)
@@
 		)
 	)
+	(polyline
+		(pts
+			(xy 284.48 41.91) (xy 222.25 41.91)
+		)
+		(stroke
+			(width 0)
+			(type default)
+		)
+	)
 	(wire
 		(pts
@@
 		)
 	)
+	(polyline
+		(pts
+			(xy 107.95 90.17) (xy 158.75 90.17)
+		)
+		(stroke
+			(width 0)
+			(type default)
+		)
+	)
 	(wire
 		(pts
@@
 		)
 	)
+	(polyline
+		(pts
+			(xy 107.95 57.15) (xy 107.95 34.29)
+		)
+		(stroke
+			(width 0)
+			(type default)
+		)
+	)
 	(wire
 		(pts
@@
 		)
 	)
+	(polyline
+		(pts
+			(xy 107.95 11.43) (xy 107.95 34.29)
+		)
+		(stroke
+			(width 0)
+			(type default)
+		)
+	)
 	(wire
 		(pts
@@
 		(pts
 			(xy 45.72 25.4) (xy 45.72 27.94)
+		)
+		(stroke
+			(width 0)
+			(type default)
+		)
+	)
+	(polyline
+		(pts
+			(xy 11.43 57.15) (xy 107.95 57.15)
 		)
 		(stroke
@@
 		)
 	)
+	(text "Power supply"
+		(exclude_from_sim no)
+		(at 79.756 33.274 0)
+		(effects
+			(font
+				(size 1.27 1.27)
+			)
+		)
+	)
 	(text "https://github.com/Casandro/time-marker"
 		(exclude_from_sim no)
@@
 		)
 	)
+	(text "Grid frequency"
+		(exclude_from_sim no)
+		(at 53.34 53.086 0)
+		(effects
+			(font
+				(size 1.27 1.27)
+			)
+		)
+	)
 	(text "Gehäuse: Industriegehäuse, 160 x 120 x 90 mm, IP66"
 		(exclude_from_sim no)
@@
 		)
 	)
+	(text "marker generator"
+		(exclude_from_sim no)
+		(at 88.138 159.512 0)
+		(effects
+			(font
+				(size 1.27 1.27)
+			)
+		)
+	)
+	(text "optional lights and switches"
+		(exclude_from_sim no)
+		(at 143.764 88.392 0)
+		(effects
+			(font
+				(size 1.27 1.27)
+			)
+		)
+	)
 	(text "Data to GNSS"
 		(exclude_from_sim no)
@@
 		(effects
 			(font
+				(size 1.27 1.27)
+			)
+		)
+	)
+	(text "optional RS232 port"
+		(exclude_from_sim no)
+		(at 196.85 157.48 0)
+		(effects
+			(font
